Commit message: With realsense

File: franka_description/robots/panda_arm.urdf.xacro (robot description, xacro)
@@ -14,3 +14,10 @@
   <xacro:include filename="$(find franka_description)/robots/panda_arm.ros2_control.xacro"/>
   <xacro:panda_arm_ros2_control ns="$(arg arm_id)" robot_ip="$(arg robot_ip)" use_fake_hardware="$(arg use_fake_hardware)" fake_sensor_commands="$(arg fake_sensor_commands)"/>
+  <xacro:property name="M_PI"              value="3.1415926535897931"/>
+	<xacro:arg      name="camera_pose_trans" default="0.02 0.0 0.055"/>
+	<xacro:arg      name="camera_pose_rot"   default="${M_PI} ${-M_PI/2.0} 0.0"/>
+    <xacro:include filename="$(find franka_description)/camera/_d435.urdf.xacro" />
+		<xacro:sensor_d435 name="camera" topics_ns="camera/" parent="panda_hand" publish_pointcloud="true">
+			<origin xyz="$(arg camera_pose_trans)" rpy="$(arg camera_pose_rot)" />
+		</xacro:sensor_d435>
 </robot>

File: franka_moveit_config/srdf/hand.xacro (robot description, xacro)
@@ -11,4 +11,6 @@
     <disable_collisions link1="${arm_id}_hand" link2="${arm_id}_leftfinger" reason="Adjacent"/>
     <disable_collisions link1="${arm_id}_hand" link2="${arm_id}_rightfinger" reason="Adjacent"/>
+    <disable_collisions link1="${arm_id}_hand" link2="camera_bottom_screw_frame" reason="Adjacent"/>
+    <disable_collisions link1="${arm_id}_hand" link2="camera_link" reason="Adjacent"/>
     <disable_collisions link1="${arm_id}_leftfinger" link2="${arm_id}_rightfinger" reason="Default"/>
   </xacro:macro>

Commit message: base plate, not in the right place

File: franka_description/robots/panda_arm.urdf.xacro (robot description, xacro)
@@ -21,3 +21,42 @@
 			<origin xyz="$(arg camera_pose_trans)" rpy="$(arg camera_pose_rot)" />
 		</xacro:sensor_d435>
+  <link name="base_plate_link">
+    <inertial>
+      <origin
+        xyz="0 0 0"
+        rpy="0 0 0" />
+      <mass
+        value="10.671" />
+      <inertia
+        ixx="0.099298"
+        ixy="-9.8583E-09"
+        ixz="-5.0395E-05"
+        iyy="0.13796"
+        iyz="-4.0684E-09"
+        izz="0.080836" />
+    </inertial>
+    <visual>
+       <!-- <origin xyz="0.57 -0.056 -0.13" rpy="0 0 1.57" /> -->
+       <origin xyz="-0.475 -0.115 0.03 " rpy="0 0 1.57" />
+       <!-- <origin xyz="-0.475 -0.115 0.065 " rpy="0 0 1.57" /> -->
+       <geometry>
+	     <mesh filename="package://franka_description/meshes/visual/base_with_top.STL"/>
+       </geometry>
+       <material name="darkgrey">
+         <color rgba="0.75294 0.75294 0.75294 1"/>
+       </material>
+    </visual>
+    <collision>
+       <!-- <origin xyz="0.57 -0.056 -0.13" rpy="0 0 1.57 " /> -->
+       <origin xyz="-0.475 -0.115 0.03 " rpy="0 0 1.57" />
+       <geometry>
+         <mesh filename="package://franka_description/meshes/visual/base_with_top.STL"/>
+       </geometry>
+    </collision>
+  </link>
+  <joint name="base_plate_joint" type="fixed">
+    <parent link="panda_link0"/>
+    <child link="base_plate_link"/>
+    <origin xyz="0.0 0.0 -0.8" rpy="0 0 0"/>
+  </joint>
 </robot>

Commit message: basplate

File: franka_description/robots/panda_arm.urdf.xacro (robot description, xacro)
@@ -58,5 +58,5 @@
     <parent link="panda_link0"/>
     <child link="base_plate_link"/>
-    <origin xyz="0.0 0.0 -0.8" rpy="0 0 0"/>
+    <origin xyz="0.21 -0.1 -0.77" rpy="0 0 0"/>
   </joint>
 </robot>

File: franka_moveit_config/srdf/panda_arm.xacro (robot description, xacro)
@@ -29,4 +29,6 @@
     <disable_collisions link1="${arm_id}_link6" link2="${arm_id}_link8" reason="Default"/>
     <disable_collisions link1="${arm_id}_link7" link2="${arm_id}_link8" reason="Adjacent"/>
+    <disable_collisions link1="${arm_id}_link0" link2="base_plate_link" reason="Never"/>
+    <disable_collisions link1="${arm_id}_link1" link2="base_plate_link" reason="Never"/>
   </xacro:macro>
 </robot>
