Commit message: hand test

File: franka_description/robots/hand.xacro (robot description, xacro)
@@ -1,6 +1,8 @@
 <?xml version="1.0" encoding="utf-8"?>
 <robot xmlns:xacro="http://www.ros.org/wiki/xacro" name="hand">
+  <xacro:arg name="use_gazebo_sim" default="false"/>
   <!-- safety_distance: Minimum safety distance in [m] by which the collision volumes are expanded and which is enforced during robot motions -->
-  <xacro:macro name="hand" params="connected_to:='' ns:='' rpy:='0 0 0' xyz:='0 0 0' safety_distance:=0">
+  <xacro:macro name="hand" params="connected_to:='' ns:='' rpy:='0 0 0' xyz:='0 0 0' safety_distance:=0
+    use_cylinder_collision_model:='false'">
     <xacro:unless value="${connected_to == ''}">
       <joint name="${ns}_hand_joint" type="fixed">
@@ -13,44 +15,121 @@
       <visual>
         <geometry>
-          <mesh filename="package://franka_description/meshes/visual/hand.dae"/>
+          <mesh filename="file://$(find franka_description)/meshes/visual/hand.dae"/>
         </geometry>
       </visual>
-      <collision>
-        <origin xyz="0 0 0.04" rpy="0 ${pi/2} ${pi/2}"/>
+      <xacro:if value="${use_cylinder_collision_model}">
+        <collision>
+          <origin xyz="0 0 0.04" rpy="0 ${pi/2} ${pi/2}"/>
+          <geometry>
+            <cylinder radius="${0.04+safety_distance}" length="0.1" />
+          </geometry>
+        </collision>
+        <collision>
+          <origin xyz="0 -0.05 0.04" rpy="0 0 0"/>
+          <geometry>
+            <sphere radius="${0.04+safety_distance}"  />
+          </geometry>
+        </collision>
+        <collision>
+          <origin xyz="0 0.05 0.04" rpy="0 0 0"/>
+          <geometry>
+            <sphere radius="${0.04+safety_distance}"  />
+          </geometry>
+        </collision>
+        <collision>
+          <origin xyz="0 0 0.1" rpy="0 ${pi/2} ${pi/2}"/>
+          <geometry>
+            <cylinder radius="${0.02+safety_distance}" length="0.1" />
+          </geometry>
+        </collision>
+        <collision>
+          <origin xyz="0 -0.05 0.1" rpy="0 0 0"/>
+          <geometry>
+            <sphere radius="${0.02+safety_distance}"  />
+          </geometry>
+        </collision>
+        <collision>
+          <origin xyz="0 0.05 0.1" rpy="0 0 0"/>
+          <geometry>
+            <sphere radius="${0.02+safety_distance}"  />
+          </geometry>
+        </collision>
+      </xacro:if>
+      <xacro:unless value="${use_cylinder_collision_model}">
+        <collision>
+          <geometry>
+            <mesh filename="file://$(find franka_description)/meshes/collision/hand.stl"/>
+          </geometry>
+        </collision>
+      </xacro:unless>
+      <xacro:if value="$(arg use_gazebo_sim)">
+        <inertial>
+          <origin xyz="0 0 0" rpy="0 0 0" />
+          <mass value="0.48" />
+          <inertia ixx="0.1" ixy="0.0" ixz="0.0" iyy="0.1" iyz="0.0" izz="0.1" />
+        </inertial>
+      </xacro:if>
+    </link>
+    <link name="${ns}_leftfinger">
+      <visual>
         <geometry>
-          <cylinder radius="${0.04+safety_distance}" length="0.1"/>
+          <mesh filename="file://$(find franka_description)/meshes/visual/finger.dae"/>
         </geometry>
-      </collision>
-      <collision>
-        <origin xyz="0 -0.05 0.04" rpy="0 0 0"/>
+      </visual>
+      <xacro:unless value="${use_cylinder_collision_model}">
+        <collision>
+          <geometry>
+            <mesh filename="file://$(find franka_description)/meshes/collision/finger.stl"/>
+          </geometry>
+        </collision>
+      </xacro:unless>
+      <xacro:if value="$(arg use_gazebo_sim)">
+        <inertial>
+          <origin xyz="0 0 0" rpy="0 0 0" />
+          <mass value="0.1" />
+          <inertia ixx="0.1" ixy="0.0" ixz="0.0" iyy="0.1" iyz="0.0" izz="0.1" />
+        </inertial>
+      </xacro:if>
+    </link>
+    <link name="${ns}_rightfinger">
+      <visual>
+        <origin xyz="0 0 0" rpy="0 0 ${pi}"/>
         <geometry>
-          <sphere radius="${0.04+safety_distance}"/>
+          <mesh filename="file://$(find franka_description)/meshes/visual/finger.dae"/>
         </geometry>
-      </collision>
-      <collision>
-        <origin xyz="0 0.05 0.04" rpy="0 0 0"/>
-        <geometry>
-          <sphere radius="${0.04+safety_distance}"/>
-        </geometry>
-      </collision>
-      <collision>
-        <origin xyz="0 0 0.1" rpy="0 ${pi/2} ${pi/2}"/>
-        <geometry>
-          <cylinder radius="${0.02+safety_distance}" length="0.1"/>
-        </geometry>
-      </collision>
-      <collision>
-        <origin xyz="0 -0.05 0.1" rpy="0 0 0"/>
-        <geometry>
-          <sphere radius="${0.02+safety_distance}"/>
-        </geometry>
-      </collision>
-      <collision>
-        <origin xyz="0 0.05 0.1" rpy="0 0 0"/>
-        <geometry>
-          <sphere radius="${0.02+safety_distance}"/>
-        </geometry>
-      </collision>
-    </link>
+      </visual>
+      <xacro:unless value="${use_cylinder_collision_model}">
+        <collision>
+          <origin xyz="0 0 0" rpy="0 0 ${pi}"/>
+          <geometry>
+            <mesh filename="file://$(find franka_description)/meshes/collision/finger.stl"/>
+          </geometry>
+        </collision>
+      </xacro:unless>
+      <xacro:if value="$(arg use_gazebo_sim)">
+        <inertial>
+          <origin xyz="0 0 0" rpy="0 0 ${pi}" />
+          <mass value="0.1" />
+          <inertia ixx="0.1" ixy="0.0" ixz="0.0" iyy="0.1" iyz="0.0" izz="0.1" />
+        </inertial>
+      </xacro:if>
+   </link>
+    <joint name="${ns}_finger_joint1" type="prismatic">
+      <parent link="${ns}_hand"/>
+      <child link="${ns}_leftfinger"/>
+      <origin xyz="0 0 0.0584" rpy="0 0 0"/>
+      <axis xyz="0 1 0"/>
+      <limit effort="150" lower="0.0" upper="0.04" velocity="0.2"/>
+    </joint>
+    <joint name="${ns}_finger_joint2" type="prismatic">
+      <parent link="${ns}_hand"/>
+      <child link="${ns}_rightfinger"/>
+      <origin xyz="0 0 0.0584" rpy="0 0 0"/>
+      <axis xyz="0 -1 0"/>
+      <limit effort="150" lower="0.0" upper="0.04" velocity="0.2"/>
+      <xacro:unless value="$(arg use_gazebo_sim)">
+        <mimic joint="${ns}_finger_joint1" />
+      </xacro:unless>
+    </joint>
     <!-- Define the hand_tcp frame -->
     <link name="${ns}_hand_tcp"/>
@@ -60,34 +139,4 @@
       <child link="${ns}_hand_tcp"/>
     </joint>
-    <link name="${ns}_leftfinger">
-      <visual>
-        <geometry>
-          <mesh filename="package://franka_description/meshes/visual/finger.dae"/>
-        </geometry>
-      </visual>
-    </link>
-    <link name="${ns}_rightfinger">
-      <visual>
-        <origin xyz="0 0 0" rpy="0 0 ${pi}"/>
-        <geometry>
-          <mesh filename="package://franka_description/meshes/visual/finger.dae"/>
-        </geometry>
-      </visual>
-    </link>
-    <joint name="${ns}_finger_joint1" type="prismatic">
-      <parent link="${ns}_hand"/>
-      <child link="${ns}_leftfinger"/>
-      <origin xyz="0 0 0.0584" rpy="0 0 0"/>
-      <axis xyz="0 1 0"/>
-      <limit effort="20" lower="0.0" upper="0.04" velocity="0.2"/>
-    </joint>
-    <joint name="${ns}_finger_joint2" type="prismatic">
-      <parent link="${ns}_hand"/>
-      <child link="${ns}_rightfinger"/>
-      <origin xyz="0 0 0.0584" rpy="0 0 0"/>
-      <axis xyz="0 -1 0"/>
-      <limit effort="20" lower="0.0" upper="0.04" velocity="0.2"/>
-      <mimic joint="${ns}_finger_joint1"/>
-    </joint>
   </xacro:macro>
 </robot>
